File: superflat.kicad_pcb (KiCad board)
At the start: 2 copper layers, 102 x 85 mm, 94 parts, among them J1 USB_C_Receptacle_USB2.0_16P, J2 Conn_01x04_Pin, J3 Conn_01x02_Pin, J4 Conn_01x05_Pin, Q1 2N7002, SW1 SW_Push, SW10 SW_Push, SW11 SW_Push, SW12 SW_Push, SW13 SW_Push, SW14 SW_Push, SW15 SW_Push, SW16 SW_Push, SW17 SW_Push, SW18 SW_Push, SW19 SW_Push, SW2 SW_Push, SW20 SW_Push, SW21 SW_Push, SW22 SW_Push, SW23 SW_Push, SW24 SW_Push, SW25 SW_Push, SW26 SW_Push, SW27 SW_Push, SW28 SW_Push, SW29 SW_Push, SW3 SW_Push, SW30 SW_Push, SW31 SW_SPDT, SW32 SW_Push, SW4 SW_Push, SW5 SW_Push, SW6 SW_Push, SW7 SW_Push, SW8 SW_Push, SW9 SW_Push, U1 nRF52840_holyiot_18010, U2 SRV05-4, U3 BQ24075RGT, U4 XC6206PxxxMR

Commit message: V2 done!
Parts:
- added J5: Conn_01x02_Pin, Connector_PinHeader_2.54mm:PinHeader_1x02_P2.54mm_Vertical, B.Cu at (46.5, 49.9)
- added J6: Conn_01x05_Pin, Connector_PinHeader_2.54mm:PinHeader_1x05_P2.54mm_Vertical, B.Cu at (43.6, 59.1)
- added Q2: 2N7002, Package_TO_SOT_SMD:SOT-23, B.Cu at (53.2, 33.6)
- added R13: 100, Resistor_SMD:R_0805_2012Metric_Pad1.20x1.40mm_HandSolder, B.Cu at (50.3, 36.0)
- added R14: 10k, Resistor_SMD:R_0805_2012Metric_Pad1.20x1.40mm_HandSolder, B.Cu at (53.2, 36.5)
- added R15: 100k, Resistor_SMD:R_0805_2012Metric_Pad1.20x1.40mm_HandSolder, B.Cu at (50.4, 32.3)
- added SW33: SW_SPDT, custom-syms:Slide, B.Cu at (52.9, 28.7)
- added SW34: SW_Push, Jumper:SolderJumper-2_P1.3mm_Open_RoundedPad1.0x1.5mm, B.Cu at (45.2, 35.2)
- added U5: nRF52840_holyiot_18010, PCM_marbastlib-various:nRF52840_holyiot_18010_HS_simple, B.Cu at (33.4, 34.8)
- J3: moved to B.Cu
- R7: moved to F.Cu
- moved J4 34.5 mm to (116.7, 30.9)
- moved C3 23.3 mm to (80.6, 46.9), turned to 90 degrees
- moved J2 23.0 mm to (88.5, 31.3)
- moved R12 22.8 mm to (94.5, 43.9), turned to -45 degrees
- moved C7 20.4 mm to (96.1, 49.5), turned to 45 degrees
- moved L2 19.9 mm to (68.6, 28.6), turned to 0 degrees
- moved D31 19.5 mm to (68.6, 30.8), turned to 0 degrees
- moved C6 19.1 mm to (94.7, 48.1), turned to 45 degrees
- moved D32 19.0 mm to (78.2, 45.0)
- moved R4 17.9 mm to (86.9, 50.1), turned to -90 degrees
- moved R11 16.8 mm to (98.0, 45.5), turned to 0 degrees
- moved R6 16.7 mm to (78.8, 49.7), turned to 180 degrees
- moved C1 15.8 mm to (69.5, 33.5), turned to 180 degrees
- moved J3 15.1 mm to (115.1, 49.9), turned to 180 degrees
- moved R7 15.0 mm to (84.0, 44.5)
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Connections:
- net Net-(J2-Pin_2) renamed D-
- J1 pad A6: Net-(J2-Pin_3) -> D+
- J1 pad B6: Net-(J2-Pin_3) -> D+
- J2 pad 3: Net-(J2-Pin_3) -> D+
- J4 pad 2: GND -> RESET1
- J4 pad 3: RESET -> Net-(J4-Pin_3)
- J4 pad 5: Net-(J4-Pin_5) -> GND
- SW32 pad 2: RESET -> RESET1
- SW4 pad MP: (no net) -> D+
- SW5 pad MP: (no net) -> GND
- SW6 pad MP: (no net) -> GND
- SW7 pad MP: (no net) -> GND
- U1 pad 2: ROW3 -> ROW5
- U1 pad 21: RESET -> RESET1
- U1 pad 24: Net-(J2-Pin_3) -> D+
- U1 pad 31: Net-(J4-Pin_4) -> Net-(J4-Pin_3)
- U1 pad 32: Net-(J4-Pin_5) -> Net-(J4-Pin_4)
- U1 pad 4: ROW5 -> ROW3
- U2 pad 6: Net-(J2-Pin_3) -> D+
Routing:
- net COL6: track 70.0 -> 196.4 mm, vias 1 -> 8
- net GND: track 182.7 -> 62.3 mm, vias 5 -> 151
- net COL5: track 91.0 -> 197.6 mm, vias 1 -> 8
- net VSENSE: track 4.00 -> 97.2 mm, vias 0 -> 4
- net D+: track 0.00 -> 87.9 mm, vias 0 -> 3
- net Net-(J2-Pin_3): track 85.0 -> 0.00 mm, vias 4 -> 0
- net SYSOFF: track 20.9 -> 102.4 mm, vias 0 -> 2
- net +BATT: track 31.1 -> 110.7 mm, vias 2 -> 4
- net COL4: track 109.8 -> 186.0 mm, vias 1 -> 6
- net ROW5: track 161.1 -> 223.7 mm, vias 6 -> 8
- net +3.3V: track 60.4 -> 120.1 mm, vias 2 -> 3
- net +5V: track 70.1 -> 123.1 mm, vias 8 -> 7
- net COL3: track 129.0 -> 172.8 mm, vias 1 -> 7
- net RESET: track 40.5 -> 0.00 mm, vias 2 -> 0
- net Net-(J4-Pin_5): track 40.5 -> 0.00 mm, vias 1 -> 0
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- added copper zone on B.Cu, net GND
- added copper zone on F.Cu, net GND
Other:
- outline, holes or cut-outs redrawn
