File: superflat.kicad_sch (KiCad schematic)
At the start: 94 parts, among them J1 USB_C_Receptacle_USB2.0_16P, J2 Conn_01x04_Pin, J3 Conn_01x02_Pin, J4 Conn_01x05_Pin, Q1 2N7002, SW1 SW_Push, SW10 SW_Push, SW11 SW_Push, SW12 SW_Push, SW13 SW_Push, SW14 SW_Push, SW15 SW_Push, SW16 SW_Push, SW17 SW_Push, SW18 SW_Push, SW19 SW_Push, SW2 SW_Push, SW20 SW_Push, SW21 SW_Push, SW22 SW_Push, SW23 SW_Push, SW24 SW_Push, SW25 SW_Push, SW26 SW_Push, SW27 SW_Push, SW28 SW_Push, SW29 SW_Push, SW3 SW_Push, SW30 SW_Push, SW31 SW_SPDT, SW32 SW_Push, SW4 SW_Push, SW5 SW_Push, SW6 SW_Push, SW7 SW_Push, SW8 SW_Push, SW9 SW_Push, U1 nRF52840_holyiot_18010, U2 SRV05-4, U3 BQ24075RGT, U4 XC6206PxxxMR

Commit message: V2 done!
Parts:
- added J5: Conn_01x02_Pin, Connector_PinHeader_2.54mm:PinHeader_1x02_P2.54mm_Vertical, symbol Connector:Conn_01x02_Pin
- added J6: Conn_01x05_Pin, Connector_PinHeader_2.54mm:PinHeader_1x05_P2.54mm_Vertical, symbol Connector:Conn_01x05_Pin
- added Q2: 2N7002, Package_TO_SOT_SMD:SOT-23, symbol Transistor_FET:2N7002
- added R13: 100, Resistor_SMD:R_0805_2012Metric_Pad1.20x1.40mm_HandSolder, symbol Device:R
- added R14: 10k, Resistor_SMD:R_0805_2012Metric_Pad1.20x1.40mm_HandSolder, symbol Device:R
- added R15: 100k, Resistor_SMD:R_0805_2012Metric_Pad1.20x1.40mm_HandSolder, symbol Device:R
- added SW33: SW_SPDT, custom-syms:Slide, symbol Switch:SW_SPDT
- added SW34: SW_Push, Jumper:SolderJumper-2_P1.3mm_Open_RoundedPad1.0x1.5mm, symbol Switch:SW_Push
- added U5: nRF52840_holyiot_18010, PCM_marbastlib-various:nRF52840_holyiot_18010_HS_simple, symbol PCM_marbastlib-various:nRF52840_holyiot_18010
Connections:
- net +3.3V: now also J6.5 (Pin_5), U5.14 (VDD_nRF)
- net +5V: now also R13.1, U5.22 (VBUS)
- net +BATT: now also J5.1 (Pin_1), R15.1
- net COL1: now also U5.36 (P0.10-LF-NFC)
- net COL2: now also U5.29 (P1.01-LF)
- net COL3: now also U5.28 (P1.03-LF)
- net COL4: now also U5.30 (P1.02-LF)
- net COL5: now also U5.5 (P1.15-LF)
- net COL6: now also U5.3 (P1.10-LF)
- net GND: now also J4.5 (Pin_5), J5.2 (Pin_2), J6.1 (Pin_1), Q2.2 (S), R14.2, SW33.3 (C), SW34.1, U5.1 (GND), U5.13 (P0.05-A), U5.25 (GND), U5.37 (GND); no longer J4.2 (Pin_2)
- net ROW1: now also U5.6 (P0.03-LF-A)
- net ROW2: now also U5.4 (P1.13-LF)
- net ROW3: now also U1.4 (P1.13-LF), U5.33 (P1.04-LF); no longer U1.2 (P1.11-LF)
- net ROW4: now also U5.34 (P1.06-LF)
- net ROW5: now also U1.2 (P1.11-LF), U5.35 (P0.09-LF-NFC); no longer U1.4 (P1.13-LF)
- net SYSOFF: now also Q2.3 (D), SW33.2 (B)
- net VSENSE: now also U5.11 (P0.31-LF-A)
- net D+: now reaches J1.A6 (D+), J1.B6 (D+), J2.3 (Pin_3), U1.24 (D+), U2.6 (IO4)
- net D+: now also U5.24 (D+)
- net D-: now reaches J1.A7 (D-), J1.B7 (D-), J2.2 (Pin_2), U1.23 (D-), U2.1 (IO1)
- net D-: now also U5.23 (D-)
- net at U1.31 (SWDCLK): now also J4.3 (Pin_3); no longer J4.4 (Pin_4)
- net at U1.32 (SWDIO): now also J4.4 (Pin_4); no longer J4.5 (Pin_5)
- net RESET renamed RESET1
- net RESET1: now also J4.2 (Pin_2); no longer J4.3 (Pin_3)
- new net: J6.3 (Pin_3), U5.31 (SWDCLK)
- new net: J6.4 (Pin_4), U5.32 (SWDIO)
- new net: R15.2, SW33.1 (A)
- new net: Q2.1 (G), R13.2, R14.1
- new net RESET2: J6.2 (Pin_2), SW34.2, U5.21 (P0.18-RESET)
- no-connect marks 38 -> 63
Other:
- note added: "Battery Control"
- note added: "Keys"
- moved on the sheet: C2, C3, D32, J2, J3, J4, Q1, R10, R11, R12, R3, R4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
