File: src/superflat.kicad_pcb (KiCad board)
At the start: 2 copper layers, 102 x 85 mm, 103 parts, among them J1 USB_C_Receptacle_USB2.0_16P, J2 Conn_01x04_Pin, J3 Conn_01x02_Pin, J4 Conn_01x05_Pin, J5 Conn_01x02_Pin, J6 Conn_01x05_Pin, Q1 2N7002, Q2 2N7002, SW1 SW_Push, SW10 SW_Push, SW11 SW_Push, SW12 SW_Push, SW13 SW_Push, SW14 SW_Push, SW15 SW_Push, SW16 SW_Push, SW17 SW_Push, SW18 SW_Push, SW19 SW_Push, SW2 SW_Push, SW20 SW_Push, SW21 SW_Push, SW22 SW_Push, SW23 SW_Push, SW24 SW_Push, SW25 SW_Push, SW26 SW_Push, SW27 SW_Push, SW28 SW_Push, SW29 SW_Push, SW3 SW_Push, SW30 SW_Push, SW31 SW_SPDT, SW32 SW_Push, SW33 SW_SPDT, SW34 SW_Push, SW4 SW_Push, SW5 SW_Push, SW6 SW_Push, SW7 SW_Push, SW8 SW_Push, SW9 SW_Push, U1 nRF52840_holyiot_18010, U2 SRV05-4, U3 BQ24075RGT, U4 XC6206PxxxMR, U5 nRF52840_holyiot_18010

Commit message: Final cleanup
Routing:
- net GND: track 62.3 -> 93.5 mm, vias 151 -> 172
- net ROW1: track 126.3 -> 124.5 mm, vias 10 -> 8
- net +5V: track 123.1 -> 121.6 mm
- net COL1: track 182.4 -> 183.9 mm
- net +BATT: track 110.7 -> 109.9 mm
- net Earth: track 34.0 -> 33.2 mm
- net +3.3V: track 120.1 -> 119.3 mm
- net Net-(D5-A): track 12.0 -> 11.4 mm
- net COL4: track 186.0 -> 186.6 mm
- net Net-(D3-A): track 6.60 -> 6.00 mm
- net Net-(J6-Pin_4): track 15.6 -> 15.1 mm
